File: hardware_v1/lm3488_dcdc.kicad_pcb (KiCad board)
At the start: 2 copper layers, 79 x 26 mm, 31 parts, among them J1 Conn_01x02, J2 Conn_01x02, J3 Conn_01x02, J4 Conn_01x02, Q1 Q_NMOS_GDS, U1 LM3488, U2 B66206B1110T001

Commit message: final touch ups and production data
Parts:
- added C14: 100n, Capacitor_SMD:C_1206_3216Metric, B.Cu at (61.9, 19.9)
- added R7: 1k, Resistor_SMD:R_1206_3216Metric, B.Cu at (61.9, 17.5)
- moved RV1 53.0 mm to (30.4, 33.9)
- moved C1 53.0 mm to (33.0, 29.9)
- moved C10 53.0 mm to (38.5, 33.9)
- moved C11 53.0 mm to (84.6, 22.2)
- moved Q1 53.0 mm to (47.4, 22.0)
- moved R4 53.0 mm to (42.2, 25.7)
- moved R6 53.0 mm to (47.4, 31.1)
- moved U1 53.0 mm to (33.0, 20.7)
- moved C12 53.0 mm to (84.5, 33.6)
- moved C13 53.0 mm to (41.0, 32.5)
- moved C2 53.0 mm to (27.0, 23.8)
- moved C3 53.0 mm to (36.6, 18.9)
- moved C4 53.0 mm to (53.6, 20.8)
- moved C5 53.0 mm to (19.8, 33.3)
- moved C6 53.0 mm to (44.6, 25.7)
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Routing:
- net Net-(R4-Pad2): track 18.4 -> 13.1 mm
- net Net-(C14-Pad2): track 5.10 -> 9.60 mm
- net +12V: track 69.6 -> 73.5 mm
- net Net-(D1-Pad2): track 13.1 -> 14.1 mm
