File: hardware_v1/lm3488_dcdc.sch (KiCad schematic (older format))
At the start: 31 parts, among them J1 Conn_01x02, J2 Conn_01x02, J3 Conn_01x02, J4 Conn_01x02, Q1 Q_NMOS_GDS, U1 LM3488, U2 B66206B1110T001

Commit message: add schematic
Parts:
- D1, D2, D3, D4: value MBRS3200T3G -> V2F22HM3/H; footprint Diode_SMD:D_SMA-SMB_Universal_Handsoldering -> Diode_SMD:D_SMF
Connections:
- net +7V: now also C10.1, C13.1, D4.1 (K); no longer C12.1, C9.1, D3.1 (K)
- net +x: now also C12.1, C9.1, D3.1 (K); no longer C10.1, C13.1, D4.1 (K)
Changed lines of the file:
@@
 Wire Wire Line
 	6650 2250 6800 2250
-Text GLabel 8600 2150 2    50   Input ~ 0
+Text GLabel 8600 3150 2    50   Input ~ 0
 +7V
 $Comp
@@
 	1    0    0    -1
 $EndComp
-Text GLabel 8600 2300 2    50   Input ~ 0
+Text GLabel 8600 3300 2    50   Input ~ 0
 FEEDBACK
 Wire Wire Line
-	8600 2300 8450 2300
-Wire Wire Line
-	8450 2300 8450 2150
-Connection ~ 8450 2150
-Wire Wire Line
-	8450 2150 8600 2150
+	8600 3300 8450 3300
+Wire Wire Line
+	8450 3300 8450 3150
+Connection ~ 8450 3150
+Wire Wire Line
+	8450 3150 8600 3150
 Text GLabel 800  3450 1    50   Input ~ 0
 FEEDBACK
@@
 	7600 3150 7600 3250
 Connection ~ 7600 3150
-Text GLabel 8600 3150 2    50   Input ~ 0
+Text GLabel 8600 2150 2    50   Input ~ 0
 +x
 $Comp
@@
 P 7350 1200
 F 0 "D2" H 7350 995 50  0000 C CNN
-F 1 "MBRS3200T3G" H 7350 1086 50  0000 C CNN
-F 2 "Diode_SMD:D_SMA-SMB_Universal_Handsoldering" V 7350 1200 50  0001 C CNN
+F 1 "V2F22HM3/H" H 7350 1086 50  0000 C CNN
+F 2 "Diode_SMD:D_SMF" V 7350 1200 50  0001 C CNN
 F 3 "~" V 7350 1200 50  0001 C CNN
 	1    7350 1200
-	-1   0    0    1
-$EndComp
-$Comp
-L Device:D_Schottky_Small D3
-U 1 1 601F0B84
-P 7350 2150
-F 0 "D3" H 7350 1945 50  0000 C CNN
-F 1 "MBRS3200T3G" H 7350 2036 50  0000 C CNN
-F 2 "Diode_SMD:D_SMA-SMB_Universal_Handsoldering" V 7350 2150 50  0001 C CNN
-F 3 "~" V 7350 2150 50  0001 C CNN
-	1    7350 2150
-	-1   0    0    1
-$EndComp
-$Comp
-L Device:D_Schottky_Small D4
-U 1 1 601F1213
-P 7350 3150
-F 0 "D4" H 7350 2945 50  0000 C CNN
-F 1 "MBRS3200T3G" H 7350 3036 50  0000 C CNN
-F 2 "Diode_SMD:D_SMA-SMB_Universal_Handsoldering" V 7350 3150 50  0001 C CNN
-F 3 "~" V 7350 3150 50  0001 C CNN
-	1    7350 3150
 	-1   0    0    1
 $EndComp
@@
 Wire Wire Line
 	8000 2250 8000 2150
-Connection ~ 8000 2150
-Wire Wire Line
-	8000 2150 8450 2150
+Wire Wire Line
+	8000 3150 8450 3150
 $Comp
 L Device:C_Small C13
@@
 Wire Wire Line
 	8000 3250 8000 3150
-Connection ~ 8000 3150
-Wire Wire Line
-	8000 3150 8600 3150
 Wire Wire Line
 	8000 3450 8000 3500
@@
 	1050 3650 2450 3650
 $Comp
-L Device:D_Schottky_Small D1
-U 1 1 6024A48B
-P 4700 1650
-F 0 "D1" V 4654 1718 50  0000 L CNN
-F 1 "MBRS3200T3G" V 4745 1718 50  0000 L CNN
-F 2 "Diode_SMD:D_SMA-SMB_Universal_Handsoldering" V 4700 1650 50  0001 C CNN
-F 3 "~" V 4700 1650 50  0001 C CNN
-	1    4700 1650
-	0    1    1    0
-$EndComp
-$Comp
 L Device:C_Small C7
 U 1 1 601429B9
@@
 	1    0    0    -1
 $EndComp
+Connection ~ 8000 3150
+Wire Wire Line
+	8600 2150 8000 2150
+Connection ~ 8000 2150
+$Comp
+L Device:D_Schottky_Small D3
+U 1 1 602A7E84
+P 7350 2150
+F 0 "D3" H 7350 1945 50  0000 C CNN
+F 1 "V2F22HM3/H" H 7350 2036 50  0000 C CNN
+F 2 "Diode_SMD:D_SMF" V 7350 2150 50  0001 C CNN
+F 3 "~" V 7350 2150 50  0001 C CNN
+	1    7350 2150
+	-1   0    0    1
+$EndComp
+$Comp
+L Device:D_Schottky_Small D4
+U 1 1 602A8151
+P 7350 3150
+F 0 "D4" H 7350 2945 50  0000 C CNN
+F 1 "V2F22HM3/H" H 7350 3036 50  0000 C CNN
+F 2 "Diode_SMD:D_SMF" V 7350 3150 50  0001 C CNN
+F 3 "~" V 7350 3150 50  0001 C CNN
+	1    7350 3150
+	-1   0    0    1
+$EndComp
+$Comp
+L Device:D_Schottky_Small D1
+U 1 1 602A8604
+P 4700 1650
+F 0 "D1" V 4654 1718 50  0000 L CNN
+F 1 "V2F22HM3/H" V 4745 1718 50  0000 L CNN
+F 2 "Diode_SMD:D_SMF" V 4700 1650 50  0001 C CNN
+F 3 "~" V 4700 1650 50  0001 C CNN
+	1    4700 1650
+	0    1    1    0
+$EndComp
 $EndSCHEMATC

Commit message: final touch ups and production data
Parts:
- added C14: 100n, Capacitor_SMD:C_1206_3216Metric, symbol Device:C_Small
- added R7: 1k, Resistor_SMD:R_1206_3216Metric, symbol Device:R_Small
Connections:
- net +12V: now also C14.1, R7.2
- net at C7.2, D1.1 (K), R5.1: now also C14.2, R7.1
Other:
- moved on the sheet: R5
Changed lines of the file:
@@
 L Device:R_Small R5
 U 1 1 60142F2A
-P 4250 1300
-F 0 "R5" H 4191 1254 50  0000 R CNN
-F 1 "1k" H 4191 1345 50  0000 R CNN
-F 2 "Resistor_SMD:R_1206_3216Metric" H 4250 1300 50  0001 C CNN
-F 3 "~" H 4250 1300 50  0001 C CNN
-	1    4250 1300
+P 4450 1250
+F 0 "R5" H 4391 1204 50  0000 R CNN
+F 1 "1k" H 4391 1295 50  0000 R CNN
+F 2 "Resistor_SMD:R_1206_3216Metric" H 4450 1250 50  0001 C CNN
+F 3 "~" H 4450 1250 50  0001 C CNN
+	1    4450 1250
 	-1   0    0    1
 $EndComp
@@
 	4700 1750 4700 1850
 Wire Wire Line
-	4250 1400 4250 1450
-Wire Wire Line
-	4250 1450 4700 1450
+	4250 1450 4450 1450
 Wire Wire Line
 	4700 1450 4700 1550
@@
 	4700 1350 4700 1450
 Wire Wire Line
-	4250 1050 4700 1050
-Wire Wire Line
-	4250 1050 4250 1200
+	4250 1050 4450 1050
 Connection ~ 4700 1050
 Wire Wire Line
@@
 	0    1    1    0
 $EndComp
+$Comp
+L Device:C_Small C14
+U 1 1 6019474C
+P 5050 1250
+F 0 "C14" H 5142 1296 50  0000 L CNN
+F 1 "100n" H 5142 1205 50  0000 L CNN
+F 2 "Capacitor_SMD:C_1206_3216Metric" H 5050 1250 50  0001 C CNN
+F 3 "~" H 5050 1250 50  0001 C CNN
+	1    5050 1250
+	1    0    0    -1
+$EndComp
+$Comp
+L Device:R_Small R7
+U 1 1 601957BF
+P 4250 1250
+F 0 "R7" H 4191 1204 50  0000 R CNN
+F 1 "1k" H 4191 1295 50  0000 R CNN
+F 2 "Resistor_SMD:R_1206_3216Metric" H 4250 1250 50  0001 C CNN
+F 3 "~" H 4250 1250 50  0001 C CNN
+	1    4250 1250
+	-1   0    0    1
+$EndComp
+Wire Wire Line
+	4450 1350 4450 1450
+Connection ~ 4450 1450
+Wire Wire Line
+	4450 1450 4700 1450
+Wire Wire Line
+	4250 1350 4250 1450
+Wire Wire Line
+	4250 1150 4250 1050
+Wire Wire Line
+	4450 1150 4450 1050
+Connection ~ 4450 1050
+Wire Wire Line
+	4450 1050 4700 1050
+Wire Wire Line
+	5050 1150 5050 1050
+Wire Wire Line
+	5050 1050 4700 1050
+Wire Wire Line
+	5050 1350 5050 1450
+Wire Wire Line
+	5050 1450 4700 1450
 $EndSCHEMATC
